Commit message: arreglando urdf

File: src/hexapod_mantis/urdf/.ipynb_checkpoints/dynamixel_hexapod-checkpoint.urdf (robot description, URDF)
Before this commit: robot dynamixel_hexapod, 20 links, 19 joints
Links:
- removed link world
- link 1A_link: geometry collision mesh filename=package://dynamixel_hexapod_description/meshes/1A_link.STL; visual mesh filename=package://dynamixel_hexapod_description/meshes/1A_link.STL
- link 1B_link: geometry collision mesh filename=package://dynamixel_hexapod_description/meshes/1B_link.STL; visual mesh filename=package://dynamixel_hexapod_description/meshes/1B_link.STL
- link 1C_link: geometry collision mesh filename=package://dynamixel_hexapod_description/meshes/1C_link.STL; visual mesh filename=package://dynamixel_hexapod_description/meshes/1C_link.STL
- link 2A_link: geometry collision mesh filename=package://dynamixel_hexapod_description/meshes/2A_link.STL; visual mesh filename=package://dynamixel_hexapod_description/meshes/2A_link.STL
- link 2B_link: geometry collision mesh filename=package://dynamixel_hexapod_description/meshes/2B_link.STL; visual mesh filename=package://dynamixel_hexapod_description/meshes/2B_link.STL
- link 2C_link: geometry collision mesh filename=package://dynamixel_hexapod_description/meshes/2C_link.STL; visual mesh filename=package://dynamixel_hexapod_description/meshes/2C_link.STL
- link 3A_link: geometry collision mesh filename=package://dynamixel_hexapod_description/meshes/3A_link.STL; visual mesh filename=package://dynamixel_hexapod_description/meshes/3A_link.STL
- link 3B_link: geometry collision mesh filename=package://dynamixel_hexapod_description/meshes/3B_link.STL; visual mesh filename=package://dynamixel_hexapod_description/meshes/3B_link.STL
- link 3C_link: geometry collision mesh filename=package://dynamixel_hexapod_description/meshes/3C_link.STL; visual mesh filename=package://dynamixel_hexapod_description/meshes/3C_link.STL
- link 4A_link: geometry collision mesh filename=package://dynamixel_hexapod_description/meshes/4A_link.STL; visual mesh filename=package://dynamixel_hexapod_description/meshes/4A_link.STL
- link 4B_link: geometry collision mesh filename=package://dynamixel_hexapod_description/meshes/4B_link.STL; visual mesh filename=package://dynamixel_hexapod_description/meshes/4B_link.STL
- link 4C_link: geometry collision mesh filename=package://dynamixel_hexapod_description/meshes/4C_link.STL; visual mesh filename=package://dynamixel_hexapod_description/meshes/4C_link.STL
- link 5A_link: geometry collision mesh filename=package://dynamixel_hexapod_description/meshes/5A_link.STL; visual mesh filename=package://dynamixel_hexapod_description/meshes/5A_link.STL
- link 5B_link: geometry collision mesh filename=package://dynamixel_hexapod_description/meshes/5B_link.STL; visual mesh filename=package://dynamixel_hexapod_description/meshes/5B_link.STL
- link 5C_link: geometry collision mesh filename=package://dynamixel_hexapod_description/meshes/5C_link.STL; visual mesh filename=package://dynamixel_hexapod_description/meshes/5C_link.STL
- link 6A_link: geometry collision mesh filename=package://dynamixel_hexapod_description/meshes/6A_link.STL; visual mesh filename=package://dynamixel_hexapod_description/meshes/6A_link.STL
- link 6B_link: geometry collision mesh filename=package://dynamixel_hexapod_description/meshes/6B_link.STL; visual mesh filename=package://dynamixel_hexapod_description/meshes/6B_link.STL
- link 6C_link: geometry collision mesh filename=package://dynamixel_hexapod_description/meshes/6C_link.STL; visual mesh filename=package://dynamixel_hexapod_description/meshes/6C_link.STL
- link base_link: geometry collision mesh filename=package://dynamixel_hexapod_description/meshes/base_link.STL; visual mesh filename=package://dynamixel_hexapod_description/meshes/base_link.STL
Joints:
- removed joint world_to_base_link
- joint 1A_joint: axis -0.013133 0 0.99991 -> 0 0 1
- joint 2A_joint: axis 0.013133 0 -0.99991 -> 0 0 1; origin xyz=0.063953 -0.10903 -0.0064656 rpy=0.091095 -0.034728 -1.0878 -> xyz=0.109 -0.62 0.03 rpy=0 0 0

File: src/hexapod_mantis/urdf/dynamixel_hexapod.urdf (robot description, URDF)
Before this commit: robot dynamixel_hexapod, 20 links, 19 joints
Links:
- removed link world
- link 1A_link: geometry collision mesh filename=package://dynamixel_hexapod_description/meshes/1A_link.STL; visual mesh filename=package://dynamixel_hexapod_description/meshes/1A_link.STL
- link 1B_link: geometry collision mesh filename=package://dynamixel_hexapod_description/meshes/1B_link.STL; visual mesh filename=package://dynamixel_hexapod_description/meshes/1B_link.STL
- link 1C_link: geometry collision mesh filename=package://dynamixel_hexapod_description/meshes/1C_link.STL; visual mesh filename=package://dynamixel_hexapod_description/meshes/1C_link.STL
- link 2A_link: geometry collision mesh filename=package://dynamixel_hexapod_description/meshes/2A_link.STL; visual mesh filename=package://dynamixel_hexapod_description/meshes/2A_link.STL
- link 2B_link: geometry collision mesh filename=package://dynamixel_hexapod_description/meshes/2B_link.STL; visual mesh filename=package://dynamixel_hexapod_description/meshes/2B_link.STL
- link 2C_link: geometry collision mesh filename=package://dynamixel_hexapod_description/meshes/2C_link.STL; visual mesh filename=package://dynamixel_hexapod_description/meshes/2C_link.STL
- link 3A_link: geometry collision mesh filename=package://dynamixel_hexapod_description/meshes/3A_link.STL; visual mesh filename=package://dynamixel_hexapod_description/meshes/3A_link.STL
- link 3B_link: geometry collision mesh filename=package://dynamixel_hexapod_description/meshes/3B_link.STL; visual mesh filename=package://dynamixel_hexapod_description/meshes/3B_link.STL
- link 3C_link: geometry collision mesh filename=package://dynamixel_hexapod_description/meshes/3C_link.STL; visual mesh filename=package://dynamixel_hexapod_description/meshes/3C_link.STL
- link 4A_link: geometry collision mesh filename=package://dynamixel_hexapod_description/meshes/4A_link.STL; visual mesh filename=package://dynamixel_hexapod_description/meshes/4A_link.STL
- link 4B_link: geometry collision mesh filename=package://dynamixel_hexapod_description/meshes/4B_link.STL; visual mesh filename=package://dynamixel_hexapod_description/meshes/4B_link.STL
- link 4C_link: geometry collision mesh filename=package://dynamixel_hexapod_description/meshes/4C_link.STL; visual mesh filename=package://dynamixel_hexapod_description/meshes/4C_link.STL
- link 5A_link: geometry collision mesh filename=package://dynamixel_hexapod_description/meshes/5A_link.STL; visual mesh filename=package://dynamixel_hexapod_description/meshes/5A_link.STL
- link 5B_link: geometry collision mesh filename=package://dynamixel_hexapod_description/meshes/5B_link.STL; visual mesh filename=package://dynamixel_hexapod_description/meshes/5B_link.STL
- link 5C_link: geometry collision mesh filename=package://dynamixel_hexapod_description/meshes/5C_link.STL; visual mesh filename=package://dynamixel_hexapod_description/meshes/5C_link.STL
- link 6A_link: geometry collision mesh filename=package://dynamixel_hexapod_description/meshes/6A_link.STL; visual mesh filename=package://dynamixel_hexapod_description/meshes/6A_link.STL
- link 6B_link: geometry collision mesh filename=package://dynamixel_hexapod_description/meshes/6B_link.STL; visual mesh filename=package://dynamixel_hexapod_description/meshes/6B_link.STL
- link 6C_link: geometry collision mesh filename=package://dynamixel_hexapod_description/meshes/6C_link.STL; visual mesh filename=package://dynamixel_hexapod_description/meshes/6C_link.STL
- link base_link: geometry collision mesh filename=package://dynamixel_hexapod_description/meshes/base_link.STL; visual mesh filename=package://dynamixel_hexapod_description/meshes/base_link.STL
Joints:
- removed joint world_to_base_link
- joint 1A_joint: origin xyz=0.109 0.062 0.03 rpy=0 0 0 -> xyz=0.12657 0 0 rpy=0.0040871 -0.089676 -0.0398
