Commit message: posicion de A

File: src/dynamixel_hexapod_description/urdf/dynamixel_hexapod.urdf (robot description, URDF)
Before this commit: robot dynamixel_hexapod, 20 links, 19 joints
Joints:
- joint 2A_joint: origin xyz=0.063953 -0.10903 -0.0064656 rpy=0.091095 -0.034728 -1.0878 -> xyz=0.109 -0.062 0.03 rpy=0 0 0
- joint 3A_joint: origin xyz=-0.061283 -0.10903 -0.019397 rpy=0.087154 0.06795 -2.1305 -> xyz=0 -0.125 0.03 rpy=0 0 0
- joint 4A_joint: origin xyz=-0.1239 0 -0.025862 rpy=-0.0040982 0.11594 3.1017 -> xyz=-0.109 -0.062 0.03 rpy=0 0 0
- joint 5A_joint: origin xyz=-0.061283 0.10903 -0.019397 rpy=-0.091209 0.060886 2.0514 -> xyz=-0.109 0.062 0.03 rpy=0 0 0
- joint 6A_joint: origin xyz=0.0639532743510104 0.109034291855445 -0.00646562448057778 rpy=-0.0870289746680175 -0.0417833420081687 1.00880226194828 -> xyz=0 0.1259 0.03 rpy=0 0 0

Commit message: urdf arreglado, falta corregir solo limites

File: src/dynamixel_hexapod_description/urdf/dynamixel_hexapod.urdf (robot description, URDF)
Before this commit: robot dynamixel_hexapod, 20 links, 19 joints
Joints:
- joint 1A_joint: origin xyz=0.109 0.062 0.03 rpy=0 0 0 -> xyz=0.109 0.062 0.03 rpy=0 0 0.523599
- joint 2A_joint: origin xyz=0.109 -0.062 0.03 rpy=0 0 0 -> xyz=0.109 -0.062 0.03 rpy=0 0 -0.525399
- joint 3A_joint: origin xyz=0 -0.125 0.03 rpy=0 0 0 -> xyz=0 -0.125 0.03 rpy=0 0 -1.5708
- joint 4A_joint: origin xyz=-0.109 -0.062 0.03 rpy=0 0 0 -> xyz=-0.109 -0.062 0.03 rpy=0 0 -2.61799
- joint 4B_joint: origin xyz=0.0782500731858154 0 0 rpy=0.00541027891423858 -0.819093279009697 0.0333518742125957 -> xyz=0.0782500731858154 0 0 rpy=0.00541027891423858 -0.819093279009697 0.033351874212595
- joint 5A_joint: origin xyz=-0.109 0.062 0.03 rpy=0 0 0 -> xyz=-0.109 0.062 0.03 rpy=0 0 -3.66519
- joint 6A_joint: origin xyz=0 0.1259 0.03 rpy=0 0 0 -> xyz=0 0.1259 0.03 rpy=0 0 1.5708

Commit message: limites corregidos

File: src/dynamixel_hexapod_description/urdf/dynamixel_hexapod.urdf (robot description, URDF)
Before this commit: robot dynamixel_hexapod, 20 links, 19 joints
Joints:
- joint 1B_joint: limit lower=-2.9671 upper=1.7453 effort=1 velocity=1 -> lower=-1.719 upper=3 effort=1 velocity=1
- joint 1C_joint: limit lower=-0.872665 upper=2.96706 effort=1 velocity=1 -> lower=-2.4 upper=1.182 effort=1 velocity=1
- joint 2B_joint: limit lower=-2.9671 upper=1.745 effort=1 velocity=1 -> lower=-1.719 upper=3 effort=1 velocity=1
- joint 2C_joint: axis 0 -1 0 -> 0 1 0; limit lower=-0.872665 upper=2.96706 effort=1 velocity=1 -> lower=-2.4 upper=1.182 effort=1 velocity=1
- joint 3B_joint: axis 0 -1 0 -> 0 1 0; limit lower=-2.9671 upper=1.745033 effort=1 velocity=1 -> lower=-1.719 upper=3 effort=1 velocity=1
- joint 3C_joint: limit lower=-0.872665 upper=2.96706 effort=1 velocity=1 -> lower=-2.4 upper=1.182 effort=1 velocity=1
- joint 4B_joint: limit lower=-2.96706 upper=1.745033 effort=1 velocity=1 -> lower=-1.719 upper=3 effort=1 velocity=1
- joint 4C_joint: limit lower=-0.872665 upper=2.96706 effort=1 velocity=1 -> lower=-2.4 upper=1.182 effort=1 velocity=1
- joint 5B_joint: limit lower=-2.9671 upper=1.745 effort=1 velocity=1 -> lower=-1.719 upper=3 effort=1 velocity=1
- joint 5C_joint: axis 0 -1 0 -> 0 1 0; limit lower=-0.87267 upper=2.9671 effort=1 velocity=1 -> lower=-2.4 upper=1.182 effort=1 velocity=1
- joint 6B_joint: limit lower=-2.96706 upper=1.74533 effort=1 velocity=1 -> lower=-1.719 upper=3 effort=1 velocity=1
- joint 6C_joint: limit lower=-0.872665 upper=2.96706 effort=1 velocity=1 -> lower=-2.4 upper=1.182 effort=1 velocity=1

Commit message: Colliders correctos

File: src/dynamixel_hexapod_description/urdf/dynamixel_hexapod.urdf (robot description, URDF)
Before this commit: robot dynamixel_hexapod, 20 links, 19 joints
Links:
- link 1A_link: geometry collision mesh filename=package://dynamixel_hexapod_description/meshes/A_collider.d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; visual mesh filename=package://dynamixel_hexapod_description/meshes/A.dae
- link 1B_link: geometry collision mesh filename=package://dynamixel_hexapod_description/meshes/B_collider.d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; visual mesh filename=package://dynamixel_hexapod_description/meshes/B.dae
- link 1C_link: geometry collision mesh filename=package://dynamixel_hexapod_description/meshes/C_collider.d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; visual mesh filename=package://dynamixel_hexapod_description/meshes/C.dae
- link 2A_link: geometry collision mesh filename=package://dynamixel_hexapod_description/meshes/A_collider.d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; visual mesh filename=package://dynamixel_hexapod_description/meshes/A.dae
- link 2B_link: geometry collision mesh filename=package://dynamixel_hexapod_description/meshes/B_collider.d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; visual mesh filename=package://dynamixel_hexapod_description/meshes/B.dae
- link 2C_link: geometry collision mesh filename=package://dynamixel_hexapod_description/meshes/C_collider.d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; visual mesh filename=package://dynamixel_hexapod_description/meshes/C.dae
- link 3A_link: geometry collision mesh filename=package://dynamixel_hexapod_description/meshes/A_collider.d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; visual mesh filename=package://dynamixel_hexapod_description/meshes/A.dae
- link 3B_link: geometry collision mesh filename=package://dynamixel_hexapod_description/meshes/B_collider.d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; visual mesh filename=package://dynamixel_hexapod_description/meshes/B.dae
- link 3C_link: geometry collision mesh filename=package://dynamixel_hexapod_description/meshes/C_collider.d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; visual mesh filename=package://dynamixel_hexapod_description/meshes/C.dae
- link 4A_link: geometry collision mesh filename=package://dynamixel_hexapod_description/meshes/A_collider.d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; visual mesh filename=package://dynamixel_hexapod_description/meshes/A.dae
- link 4B_link: geometry collision mesh filename=package://dynamixel_hexapod_description/meshes/B_collider.d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; visual mesh filename=package://dynamixel_hexapod_description/meshes/B.dae
- link 4C_link: geometry collision mesh filename=package://dynamixel_hexapod_description/meshes/C_collider.d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; visual mesh filename=package://dynamixel_hexapod_description/meshes/C.dae
- link 5A_link: geometry collision mesh filename=package://dynamixel_hexapod_description/meshes/A_collider.d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; visual mesh filename=package://dynamixel_hexapod_description/meshes/A.dae
- link 5B_link: geometry collision mesh filename=package://dynamixel_hexapod_description/meshes/B_collider.d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; visual mesh filename=package://dynamixel_hexapod_description/meshes/B.dae
- link 5C_link: geometry collision mesh filename=package://dynamixel_hexapod_description/meshes/C_collider.d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; visual mesh filename=package://dynamixel_hexapod_description/meshes/C.dae
- link 6A_link: geometry collision mesh filename=package://dynamixel_hexapod_description/meshes/A_collider.d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; visual mesh filename=package://dynamixel_hexapod_description/meshes/A.dae
- link 6B_link: geometry collision mesh filename=package://dynamixel_hexapod_description/meshes/B_collider.d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; visual mesh filename=package://dynamixel_hexapod_description/meshes/B.dae
- link 6C_link: geometry collision mesh filename=package://dynamixel_hexapod_description/meshes/C_collider.d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; visual mesh filename=package://dynamixel_hexapod_description/meshes/C.dae
- link base_link: geometry collision mesh filename=package://dynamixel_hexapod_description/meshes/base_collide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; visual mesh filename=package://dynamixel_hexapod_description/meshes/base.dae

Commit message: primer avance en moveit, falta solucionar algunos errores

File: src/dynamixel_hexapod_description/urdf/dynamixel_hexapod.urdf (robot description, URDF)
Before this commit: robot dynamixel_hexapod, 20 links, 19 joints
Links:
- removed link world
Joints:
- removed joint world_to_base_link
