Commit message: renombrar todos los joints del proyecto joint_XA

File: src/dynamixel_hexapod_description/urdf/dynamixel_hexapod.urdf (robot description, URDF)
Before this commit: robot dynamixel_hexapod, 19 links, 18 joints
Joints:
- removed joint 1A_joint
- removed joint 1B_joint
- removed joint 1C_joint
- removed joint 2A_joint
- removed joint 2B_joint
- removed joint 2C_joint
- removed joint 3A_joint
- removed joint 3B_joint
- removed joint 3C_joint
- removed joint 4A_joint
- removed joint 4B_joint
- removed joint 4C_joint
- removed joint 5A_joint
- removed joint 5B_joint
- removed joint 5C_joint
- removed joint 6A_joint
- removed joint 6B_joint
- removed joint 6C_joint
- added joint joint_1A: type revolute, parent base_link, child 1A_link, origin xyz=0.109 0.062 0.03 rpy=0 0 0.523599, axis -0.013133 0 0.99991, limit lower=-1.5708 upper=1.5708 effort=1 velocity=1
- added joint joint_1B: type revolute, parent 1A_link, child 1B_link, origin xyz=0.07825 0 0 rpy=0.0054103 -0.81909 0.033352, axis 0 1 0, limit lower=-1.719 upper=3 effort=1 velocity=1
- added joint joint_1C: type revolute, parent 1B_link, child 1C_link, origin xyz=0.172821824222266 -0.00859357288230811 0 rpy=-3.13913475006377 1.07013691482246 -3.13476958627829, axis 0 1 0, limit lower=-2.4 upper=1.182 effort=1 velocity=1
- added joint joint_2A: type revolute, parent base_link, child 2A_link, origin xyz=0.109 -0.062 0.03 rpy=0 0 -0.525399, axis 0.013133 0 -0.99991, limit lower=-1.5708 upper=1.5708 effort=1 velocity=1
- added joint joint_2B: type revolute, parent 2A_link, child 2B_link, origin xyz=0.0782500731858153 0 0 rpy=0.00541027891423811 -0.819093279009694 0.0333518742125984, axis 0 1 0, limit lower=-1.719 upper=3 effort=1 velocity=1
- added joint joint_2C: type revolute, parent 2B_link, child 2C_link, origin xyz=0.172821824222266 -0.00859357288230778 0 rpy=-3.13913475006377 1.07013691482246 -3.13476958627829, axis 0 1 0, limit lower=-2.4 upper=1.182 effort=1 velocity=1
- added joint joint_3A: type revolute, parent base_link, child 3A_link, origin xyz=0 -0.125 0.03 rpy=0 0 -1.5708, axis -0.013133 0 0.99991, limit lower=-1.5708 upper=1.5708 effort=1 velocity=1
- added joint joint_3B: type revolute, parent 3A_link, child 3B_link, origin xyz=0.0782500731858156 0 0 rpy=0.00541027891423802 -0.819093279009695 0.0333518742125869, axis 0 1 0, limit lower=-1.719 upper=3 effort=1 velocity=1
- added joint joint_3C: type revolute, parent 3B_link, child 3C_link, origin xyz=0.172821824222266 -0.00859357288230712 0 rpy=-3.13913475006378 1.07013691482246 -3.1347695862783, axis 0 1 0, limit lower=-2.4 upper=1.182 effort=1 velocity=1
- added joint joint_4A: type revolute, parent base_link, child 4A_link, origin xyz=-0.109 -0.062 0.03 rpy=0 0 -2.61799, axis 0.013133 0 -0.99991, limit lower=-1.5708 upper=1.5708 effort=1 velocity=1
- added joint joint_4B: type revolute, parent 4A_link, child 4B_link, origin xyz=0.0782500731858154 0 0 rpy=0.00541027891423858 -0.819093279009697 0.033351874212595, axis 0 1 0, limit lower=-1.719 upper=3 effort=1 velocity=1
- added joint joint_4C: type revolute, parent 4B_link, child 4C_link, origin xyz=0.172821824222266 -0.00859357288230733 0 rpy=-3.13913475006377 1.07013691482246 -3.13476958627829, axis 0 1 0, limit lower=-2.4 upper=1.182 effort=1 velocity=1
- added joint joint_5A: type revolute, parent base_link, child 5A_link, origin xyz=-0.109 0.062 0.03 rpy=0 0 -3.66519, axis -0.013133 0 0.99991, limit lower=-1.5708 upper=1.5708 effort=1 velocity=1
- added joint joint_5B: type revolute, parent 5A_link, child 5B_link, origin xyz=0.0782500731858156 0 0 rpy=0.0054102789142378 -0.819093279009694 0.033351874212598, axis 0 1 0, limit lower=-1.719 upper=3 effort=1 velocity=1
- added joint joint_5C: type revolute, parent 5B_link, child 5C_link, origin xyz=0.172821824222266 -0.00859357288230722 0 rpy=-3.13913475006377 1.07013691482246 -3.1347695862783, axis 0 1 0, limit lower=-2.4 upper=1.182 effort=1 velocity=1
- added joint joint_6A: type revolute, parent base_link, child 6A_link, origin xyz=0 0.1259 0.03 rpy=0 0 1.5708, axis 0.0131329106165465 0 -0.999913759610667, limit lower=-1.5708 upper=1.5708 effort=1 velocity=1
- added joint joint_6B: type revolute, parent 6A_link, child 6B_link, origin xyz=0.0782500731858157 0 0 rpy=0.00541027891423497 -0.819093279009694 0.0333518742125941, axis 0 1 0, limit lower=-1.719 upper=3 effort=1 velocity=1
- added joint joint_6C: type revolute, parent 6B_link, child 6C_link, origin xyz=0.172821824222266 -0.00859357288230794 0 rpy=-3.13913475006377 1.07013691482246 -3.1347695862783, axis 0 1 0, limit lower=-2.4 upper=1.182 effort=1 velocity=1

File: src/hexapod_mantis/urdf/.ipynb_checkpoints/dynamixel_hexapod-checkpoint.urdf (robot description, URDF)
Before this commit: robot dynamixel_hexapod, 19 links, 18 joints
Joints:
- removed joint 1A_joint
- removed joint 1B_joint
- removed joint 1C_joint
- removed joint 2A_joint
- removed joint 2B_joint
- removed joint 2C_joint
- removed joint 3A_joint
- removed joint 3B_joint
- removed joint 3C_joint
- removed joint 4A_joint
- removed joint 4B_joint
- removed joint 4C_joint
- removed joint 5A_joint
- removed joint 5B_joint
- removed joint 5C_joint
- removed joint 6A_joint
- removed joint 6B_joint
- removed joint 6C_joint
- added joint joint_1A: type revolute, parent base_link, child 1A_link, origin xyz=0.109 0.062 0.03 rpy=0 0 0, axis 0 0 1, limit lower=-1.5708 upper=1.5708 effort=1 velocity=1
- added joint joint_1B: type revolute, parent 1A_link, child 1B_link, origin xyz=0.07825 0 0 rpy=0.0054103 -0.81909 0.033352, axis 0 1 0, limit lower=-2.9671 upper=1.7453 effort=1 velocity=1
- added joint joint_1C: type revolute, parent 1B_link, child 1C_link, origin xyz=0.172821824222266 -0.00859357288230811 0 rpy=-3.13913475006377 1.07013691482246 -3.13476958627829, axis 0 1 0, limit lower=-0.872665 upper=2.96706 effort=1 velocity=1
- added joint joint_2A: type revolute, parent base_link, child 2A_link, origin xyz=0.109 -0.62 0.03 rpy=0 0 0, axis 0 0 1, limit lower=-1.5708 upper=1.5708 effort=1 velocity=1
- added joint joint_2B: type revolute, parent 2A_link, child 2B_link, origin xyz=0.0782500731858153 0 0 rpy=0.00541027891423811 -0.819093279009694 0.0333518742125984, axis 0 1 0, limit lower=-2.9671 upper=1.745 effort=1 velocity=1
- added joint joint_2C: type revolute, parent 2B_link, child 2C_link, origin xyz=0.172821824222266 -0.00859357288230778 0 rpy=-3.13913475006377 1.07013691482246 -3.13476958627829, axis 0 -1 0, limit lower=-0.872665 upper=2.96706 effort=1 velocity=1
- added joint joint_3A: type revolute, parent base_link, child 3A_link, origin xyz=-0.061283 -0.10903 -0.019397 rpy=0.087154 0.06795 -2.1305, axis -0.013133 0 0.99991, limit lower=-1.5708 upper=1.5708 effort=1 velocity=1
- added joint joint_3B: type revolute, parent 3A_link, child 3B_link, origin xyz=0.0782500731858156 0 0 rpy=0.00541027891423802 -0.819093279009695 0.0333518742125869, axis 0 -1 0, limit lower=-2.9671 upper=1.745033 effort=1 velocity=1
- added joint joint_3C: type revolute, parent 3B_link, child 3C_link, origin xyz=0.172821824222266 -0.00859357288230712 0 rpy=-3.13913475006378 1.07013691482246 -3.1347695862783, axis 0 1 0, limit lower=-0.872665 upper=2.96706 effort=1 velocity=1
- added joint joint_4A: type revolute, parent base_link, child 4A_link, origin xyz=-0.1239 0 -0.025862 rpy=-0.0040982 0.11594 3.1017, axis 0.013133 0 -0.99991, limit lower=-1.5708 upper=1.5708 effort=1 velocity=1
- added joint joint_4B: type revolute, parent 4A_link, child 4B_link, origin xyz=0.0782500731858154 0 0 rpy=0.00541027891423858 -0.819093279009697 0.0333518742125957, axis 0 1 0, limit lower=-2.96706 upper=1.745033 effort=1 velocity=1
- added joint joint_4C: type revolute, parent 4B_link, child 4C_link, origin xyz=0.172821824222266 -0.00859357288230733 0 rpy=-3.13913475006377 1.07013691482246 -3.13476958627829, axis 0 1 0, limit lower=-0.872665 upper=2.96706 effort=1 velocity=1
- added joint joint_5A: type revolute, parent base_link, child 5A_link, origin xyz=-0.061283 0.10903 -0.019397 rpy=-0.091209 0.060886 2.0514, axis -0.013133 0 0.99991, limit lower=-1.5708 upper=1.5708 effort=1 velocity=1
- added joint joint_5B: type revolute, parent 5A_link, child 5B_link, origin xyz=0.0782500731858156 0 0 rpy=0.0054102789142378 -0.819093279009694 0.033351874212598, axis 0 1 0, limit lower=-2.9671 upper=1.745 effort=1 velocity=1
- added joint joint_5C: type revolute, parent 5B_link, child 5C_link, origin xyz=0.172821824222266 -0.00859357288230722 0 rpy=-3.13913475006377 1.07013691482246 -3.1347695862783, axis 0 -1 0, limit lower=-0.87267 upper=2.9671 effort=1 velocity=1
- added joint joint_6A: type revolute, parent base_link, child 6A_link, origin xyz=0.0639532743510104 0.109034291855445 -0.00646562448057778 rpy=-0.0870289746680175 -0.0417833420081687 1.00880226194828, axis 0.0131329106165465 0 -0.999913759610667, limit lower=-1.5708 upper=1.5708 effort=1 velocity=1
- added joint joint_6B: type revolute, parent 6A_link, child 6B_link, origin xyz=0.0782500731858157 0 0 rpy=0.00541027891423497 -0.819093279009694 0.0333518742125941, axis 0 1 0, limit lower=-2.96706 upper=1.74533 effort=1 velocity=1
- added joint joint_6C: type revolute, parent 6B_link, child 6C_link, origin xyz=0.172821824222266 -0.00859357288230794 0 rpy=-3.13913475006377 1.07013691482246 -3.1347695862783, axis 0 1 0, limit lower=-0.872665 upper=2.96706 effort=1 velocity=1

File: src/hexapod_mantis/urdf/dyna_hexa.urdf (robot description, URDF)
Before this commit: robot dynamixel_hexapod, 19 links, 18 joints
Joints:
- removed joint 1A_joint
- removed joint 1B_joint
- removed joint 1C_joint
- removed joint 2A_joint
- removed joint 2B_joint
- removed joint 2C_joint
- removed joint 3A_joint
- removed joint 3B_joint
- removed joint 3C_joint
- removed joint 4A_joint
- removed joint 4B_joint
- removed joint 4C_joint
- removed joint 5A_joint
- removed joint 5B_joint
- removed joint 5C_joint
- removed joint 6A_joint
- removed joint 6B_joint
- removed joint 6C_joint
- added joint joint_1A: type revolute, parent base_link, child 1A_link, origin xyz=0.12657 0 0 rpy=0.0040871 -0.089676 -0.0398, axis -0.013133 0 0.99991, limit lower=-1.5708 upper=1.5708 effort=1 velocity=1
- added joint joint_1B: type revolute, parent 1A_link, child 1B_link, origin xyz=0.07825 0 0 rpy=0.0054103 -0.81909 0.033352, axis 0 1 0, limit lower=-2.9671 upper=1.7453 effort=1 velocity=1
- added joint joint_1C: type revolute, parent 1B_link, child 1C_link, origin xyz=0.172821824222266 -0.00859357288230811 0 rpy=-3.13913475006377 1.07013691482246 -3.13476958627829, axis 0 1 0, limit lower=-0.872665 upper=2.96706 effort=1 velocity=1
- added joint joint_2A: type revolute, parent base_link, child 2A_link, origin xyz=0.063953 -0.10903 -0.0064656 rpy=0.091095 -0.034728 -1.0878, axis 0.013133 0 -0.99991, limit lower=-1.5708 upper=1.5708 effort=1 velocity=1
- added joint joint_2B: type revolute, parent 2A_link, child 2B_link, origin xyz=0.0782500731858153 0 0 rpy=0.00541027891423811 -0.819093279009694 0.0333518742125984, axis 0 1 0, limit lower=-2.9671 upper=1.745 effort=1 velocity=1
- added joint joint_2C: type revolute, parent 2B_link, child 2C_link, origin xyz=0.172821824222266 -0.00859357288230778 0 rpy=-3.13913475006377 1.07013691482246 -3.13476958627829, axis 0 -1 0, limit lower=-0.872665 upper=2.96706 effort=1 velocity=1
- added joint joint_3A: type revolute, parent base_link, child 3A_link, origin xyz=-0.061283 -0.10903 -0.019397 rpy=0.087154 0.06795 -2.1305, axis -0.013133 0 0.99991, limit lower=-1.5708 upper=1.5708 effort=1 velocity=1
- added joint joint_3B: type revolute, parent 3A_link, child 3B_link, origin xyz=0.0782500731858156 0 0 rpy=0.00541027891423802 -0.819093279009695 0.0333518742125869, axis 0 -1 0, limit lower=-2.9671 upper=1.745033 effort=1 velocity=1
- added joint joint_3C: type revolute, parent 3B_link, child 3C_link, origin xyz=0.172821824222266 -0.00859357288230712 0 rpy=-3.13913475006378 1.07013691482246 -3.1347695862783, axis 0 1 0, limit lower=-0.872665 upper=2.96706 effort=1 velocity=1
- added joint joint_4A: type revolute, parent base_link, child 4A_link, origin xyz=-0.1239 0 -0.025862 rpy=-0.0040982 0.11594 3.1017, axis 0.013133 0 -0.99991, limit lower=-1.5708 upper=1.5708 effort=1 velocity=1
- added joint joint_4B: type revolute, parent 4A_link, child 4B_link, origin xyz=0.0782500731858154 0 0 rpy=0.00541027891423858 -0.819093279009697 0.0333518742125957, axis 0 1 0, limit lower=-2.96706 upper=1.745033 effort=1 velocity=1
- added joint joint_4C: type revolute, parent 4B_link, child 4C_link, origin xyz=0.172821824222266 -0.00859357288230733 0 rpy=-3.13913475006377 1.07013691482246 -3.13476958627829, axis 0 1 0, limit lower=-0.872665 upper=2.96706 effort=1 velocity=1
- added joint joint_5A: type revolute, parent base_link, child 5A_link, origin xyz=-0.061283 0.10903 -0.019397 rpy=-0.091209 0.060886 2.0514, axis -0.013133 0 0.99991, limit lower=-1.5708 upper=1.5708 effort=1 velocity=1
- added joint joint_5B: type revolute, parent 5A_link, child 5B_link, origin xyz=0.0782500731858156 0 0 rpy=0.0054102789142378 -0.819093279009694 0.033351874212598, axis 0 1 0, limit lower=-2.9671 upper=1.745 effort=1 velocity=1
- added joint joint_5C: type revolute, parent 5B_link, child 5C_link, origin xyz=0.172821824222266 -0.00859357288230722 0 rpy=-3.13913475006377 1.07013691482246 -3.1347695862783, axis 0 -1 0, limit lower=-0.87267 upper=2.9671 effort=1 velocity=1
- added joint joint_6A: type revolute, parent base_link, child 6A_link, origin xyz=0.0639532743510104 0.109034291855445 -0.00646562448057778 rpy=-0.0870289746680175 -0.0417833420081687 1.00880226194828, axis 0.0131329106165465 0 -0.999913759610667, limit lower=-1.5708 upper=1.5708 effort=1 velocity=1
- added joint joint_6B: type revolute, parent 6A_link, child 6B_link, origin xyz=0.0782500731858157 0 0 rpy=0.00541027891423497 -0.819093279009694 0.0333518742125941, axis 0 1 0, limit lower=-2.96706 upper=1.74533 effort=1 velocity=1
- added joint joint_6C: type revolute, parent 6B_link, child 6C_link, origin xyz=0.172821824222266 -0.00859357288230794 0 rpy=-3.13913475006377 1.07013691482246 -3.1347695862783, axis 0 1 0, limit lower=-0.872665 upper=2.96706 effort=1 velocity=1

File: src/hexapod_mantis/urdf/dynamixel_hexapod.urdf (robot description, URDF)
Before this commit: robot dynamixel_hexapod, 19 links, 18 joints
Joints:
- removed joint 1A_joint
- removed joint 1B_joint
- removed joint 1C_joint
- removed joint 2A_joint
- removed joint 2B_joint
- removed joint 2C_joint
- removed joint 3A_joint
- removed joint 3B_joint
- removed joint 3C_joint
- removed joint 4A_joint
- removed joint 4B_joint
- removed joint 4C_joint
- removed joint 5A_joint
- removed joint 5B_joint
- removed joint 5C_joint
- removed joint 6A_joint
- removed joint 6B_joint
- removed joint 6C_joint
- added joint joint_1A: type revolute, parent base_link, child 1A_link, origin xyz=0.12657 0 0 rpy=0.0040871 -0.089676 -0.0398, axis -0.013133 0 0.99991, limit lower=-1.5708 upper=1.5708 effort=1 velocity=1
- added joint joint_1B: type revolute, parent 1A_link, child 1B_link, origin xyz=0.07825 0 0 rpy=0.0054103 -0.81909 0.033352, axis 0 1 0, limit lower=-2.9671 upper=1.7453 effort=1 velocity=1
- added joint joint_1C: type revolute, parent 1B_link, child 1C_link, origin xyz=0.172821824222266 -0.00859357288230811 0 rpy=-3.13913475006377 1.07013691482246 -3.13476958627829, axis 0 1 0, limit lower=-0.872665 upper=2.96706 effort=1 velocity=1
- added joint joint_2A: type revolute, parent base_link, child 2A_link, origin xyz=0.063953 -0.10903 -0.0064656 rpy=0.091095 -0.034728 -1.0878, axis 0.013133 0 -0.99991, limit lower=-1.5708 upper=1.5708 effort=1 velocity=1
- added joint joint_2B: type revolute, parent 2A_link, child 2B_link, origin xyz=0.0782500731858153 0 0 rpy=0.00541027891423811 -0.819093279009694 0.0333518742125984, axis 0 1 0, limit lower=-2.9671 upper=1.745 effort=1 velocity=1
- added joint joint_2C: type revolute, parent 2B_link, child 2C_link, origin xyz=0.172821824222266 -0.00859357288230778 0 rpy=-3.13913475006377 1.07013691482246 -3.13476958627829, axis 0 -1 0, limit lower=-0.872665 upper=2.96706 effort=1 velocity=1
- added joint joint_3A: type revolute, parent base_link, child 3A_link, origin xyz=-0.061283 -0.10903 -0.019397 rpy=0.087154 0.06795 -2.1305, axis -0.013133 0 0.99991, limit lower=-1.5708 upper=1.5708 effort=1 velocity=1
- added joint joint_3B: type revolute, parent 3A_link, child 3B_link, origin xyz=0.0782500731858156 0 0 rpy=0.00541027891423802 -0.819093279009695 0.0333518742125869, axis 0 -1 0, limit lower=-2.9671 upper=1.745033 effort=1 velocity=1
- added joint joint_3C: type revolute, parent 3B_link, child 3C_link, origin xyz=0.172821824222266 -0.00859357288230712 0 rpy=-3.13913475006378 1.07013691482246 -3.1347695862783, axis 0 1 0, limit lower=-0.872665 upper=2.96706 effort=1 velocity=1
- added joint joint_4A: type revolute, parent base_link, child 4A_link, origin xyz=-0.1239 0 -0.025862 rpy=-0.0040982 0.11594 3.1017, axis 0.013133 0 -0.99991, limit lower=-1.5708 upper=1.5708 effort=1 velocity=1
- added joint joint_4B: type revolute, parent 4A_link, child 4B_link, origin xyz=0.0782500731858154 0 0 rpy=0.00541027891423858 -0.819093279009697 0.0333518742125957, axis 0 1 0, limit lower=-2.96706 upper=1.745033 effort=1 velocity=1
- added joint joint_4C: type revolute, parent 4B_link, child 4C_link, origin xyz=0.172821824222266 -0.00859357288230733 0 rpy=-3.13913475006377 1.07013691482246 -3.13476958627829, axis 0 1 0, limit lower=-0.872665 upper=2.96706 effort=1 velocity=1
- added joint joint_5A: type revolute, parent base_link, child 5A_link, origin xyz=-0.061283 0.10903 -0.019397 rpy=-0.091209 0.060886 2.0514, axis -0.013133 0 0.99991, limit lower=-1.5708 upper=1.5708 effort=1 velocity=1
- added joint joint_5B: type revolute, parent 5A_link, child 5B_link, origin xyz=0.0782500731858156 0 0 rpy=0.0054102789142378 -0.819093279009694 0.033351874212598, axis 0 1 0, limit lower=-2.9671 upper=1.745 effort=1 velocity=1
- added joint joint_5C: type revolute, parent 5B_link, child 5C_link, origin xyz=0.172821824222266 -0.00859357288230722 0 rpy=-3.13913475006377 1.07013691482246 -3.1347695862783, axis 0 -1 0, limit lower=-0.87267 upper=2.9671 effort=1 velocity=1
- added joint joint_6A: type revolute, parent base_link, child 6A_link, origin xyz=0.0639532743510104 0.109034291855445 -0.00646562448057778 rpy=-0.0870289746680175 -0.0417833420081687 1.00880226194828, axis 0.0131329106165465 0 -0.999913759610667, limit lower=-1.5708 upper=1.5708 effort=1 velocity=1
- added joint joint_6B: type revolute, parent 6A_link, child 6B_link, origin xyz=0.0782500731858157 0 0 rpy=0.00541027891423497 -0.819093279009694 0.0333518742125941, axis 0 1 0, limit lower=-2.96706 upper=1.74533 effort=1 velocity=1
- added joint joint_6C: type revolute, parent 6B_link, child 6C_link, origin xyz=0.172821824222266 -0.00859357288230794 0 rpy=-3.13913475006377 1.07013691482246 -3.1347695862783, axis 0 1 0, limit lower=-0.872665 upper=2.96706 effort=1 velocity=1
