Commit message: renombrar todos los joints del proyecto joint_XA

File: src/moveit_config/config/dynamixel_hexapod.ros2_control.xacro (robot description, xacro)
@@ -8,127 +8,127 @@
                 <plugin>mock_components/GenericSystem</plugin>
             </hardware>
-            <joint name="1A_joint">
+            <joint name="joint_1A">
                 <command_interface name="position"/>
                 <state_interface name="position">
-                  <param name="initial_value">${initial_positions['1A_joint']}</param>
+                  <param name="initial_value">${initial_positions['joint_1A']}</param>
                 </state_interface>
                 <state_interface name="velocity"/>
             </joint>
-            <joint name="1B_joint">
+            <joint name="joint_1B">
                 <command_interface name="position"/>
                 <state_interface name="position">
-                  <param name="initial_value">${initial_positions['1B_joint']}</param>
+                  <param name="initial_value">${initial_positions['joint_1B']}</param>
                 </state_interface>
                 <state_interface name="velocity"/>
             </joint>
-            <joint name="1C_joint">
+            <joint name="joint_1C">
                 <command_interface name="position"/>
                 <state_interface name="position">
-                  <param name="initial_value">${initial_positions['1C_joint']}</param>
+                  <param name="initial_value">${initial_positions['joint_1C']}</param>
                 </state_interface>
                 <state_interface name="velocity"/>
             </joint>
-            <joint name="2A_joint">
+            <joint name="joint_2A">
                 <command_interface name="position"/>
                 <state_interface name="position">
-                  <param name="initial_value">${initial_positions['2A_joint']}</param>
+                  <param name="initial_value">${initial_positions['joint_2A']}</param>
                 </state_interface>
                 <state_interface name="velocity"/>
             </joint>
-            <joint name="2B_joint">
+            <joint name="joint_2B">
                 <command_interface name="position"/>
                 <state_interface name="position">
-                  <param name="initial_value">${initial_positions['2B_joint']}</param>
+                  <param name="initial_value">${initial_positions['joint_2B']}</param>
                 </state_interface>
                 <state_interface name="velocity"/>
             </joint>
-            <joint name="2C_joint">
+            <joint name="joint_2C">
                 <command_interface name="position"/>
                 <state_interface name="position">
-                  <param name="initial_value">${initial_positions['2C_joint']}</param>
+                  <param name="initial_value">${initial_positions['joint_2C']}</param>
                 </state_interface>
                 <state_interface name="velocity"/>
             </joint>
-            <joint name="3A_joint">
+            <joint name="joint_3A">
                 <command_interface name="position"/>
                 <state_interface name="position">
-                  <param name="initial_value">${initial_positions['3A_joint']}</param>
+                  <param name="initial_value">${initial_positions['joint_3A']}</param>
                 </state_interface>
                 <state_interface name="velocity"/>
             </joint>
-            <joint name="3B_joint">
+            <joint name="joint_3B">
                 <command_interface name="position"/>
                 <state_interface name="position">
-                  <param name="initial_value">${initial_positions['3B_joint']}</param>
+                  <param name="initial_value">${initial_positions['joint_3B']}</param>
                 </state_interface>
                 <state_interface name="velocity"/>
             </joint>
-            <joint name="3C_joint">
+            <joint name="joint_3C">
                 <command_interface name="position"/>
                 <state_interface name="position">
-                  <param name="initial_value">${initial_positions['3C_joint']}</param>
+                  <param name="initial_value">${initial_positions['joint_3C']}</param>
                 </state_interface>
                 <state_interface name="velocity"/>
             </joint>
-            <joint name="4A_joint">
+            <joint name="joint_4A">
                 <command_interface name="position"/>
                 <state_interface name="position">
-                  <param name="initial_value">${initial_positions['4A_joint']}</param>
+                  <param name="initial_value">${initial_positions['joint_4A']}</param>
                 </state_interface>
                 <state_interface name="velocity"/>
             </joint>
-            <joint name="4B_joint">
+            <joint name="joint_4B">
                 <command_interface name="position"/>
                 <state_interface name="position">
-                  <param name="initial_value">${initial_positions['4B_joint']}</param>
+                  <param name="initial_value">${initial_positions['joint_4B']}</param>
                 </state_interface>
                 <state_interface name="velocity"/>
             </joint>
-            <joint name="4C_joint">
+            <joint name="joint_4C">
                 <command_interface name="position"/>
                 <state_interface name="position">
-                  <param name="initial_value">${initial_positions['4C_joint']}</param>
+                  <param name="initial_value">${initial_positions['joint_4C']}</param>
                 </state_interface>
                 <state_interface name="velocity"/>
             </joint>
-            <joint name="5A_joint">
+            <joint name="joint_5A">
                 <command_interface name="position"/>
                 <state_interface name="position">
-                  <param name="initial_value">${initial_positions['5A_joint']}</param>
+                  <param name="initial_value">${initial_positions['joint_5A']}</param>
                 </state_interface>
                 <state_interface name="velocity"/>
             </joint>
-            <joint name="5B_joint">
+            <joint name="joint_5B">
                 <command_interface name="position"/>
                 <state_interface name="position">
-                  <param name="initial_value">${initial_positions['5B_joint']}</param>
+                  <param name="initial_value">${initial_positions['joint_5B']}</param>
                 </state_interface>
                 <state_interface name="velocity"/>
             </joint>
-            <joint name="5C_joint">
+            <joint name="joint_5C">
                 <command_interface name="position"/>
                 <state_interface name="position">
-                  <param name="initial_value">${initial_positions['5C_joint']}</param>
+                  <param name="initial_value">${initial_positions['joint_5C']}</param>
                 </state_interface>
                 <state_interface name="velocity"/>
             </joint>
-            <joint name="6A_joint">
+            <joint name="joint_6A">
                 <command_interface name="position"/>
                 <state_interface name="position">
-                  <param name="initial_value">${initial_positions['6A_joint']}</param>
+                  <param name="initial_value">${initial_positions['joint_6A']}</param>
                 </state_interface>
                 <state_interface name="velocity"/>
             </joint>
-            <joint name="6B_joint">
+            <joint name="joint_6B">
                 <command_interface name="position"/>
                 <state_interface name="position">
-                  <param name="initial_value">${initial_positions['6B_joint']}</param>
+                  <param name="initial_value">${initial_positions['joint_6B']}</param>
                 </state_interface>
                 <state_interface name="velocity"/>
             </joint>
-            <joint name="6C_joint">
+            <joint name="joint_6C">
                 <command_interface name="position"/>
                 <state_interface name="position">
-                  <param name="initial_value">${initial_positions['6C_joint']}</param>
+                  <param name="initial_value">${initial_positions['joint_6C']}</param>
                 </state_interface>
                 <state_interface name="velocity"/>

Commit message: aceleración de la siluacion en webots modificando joint_limits.yaml y dynamixel_hexapod.urdf

File: src/dynamixel_hexapod_description/urdf/dynamixel_hexapod.urdf (robot description, URDF)
Before this commit: robot dynamixel_hexapod, 19 links, 18 joints
Joints:
- joint joint_1A: limit lower=-1.5708 upper=1.5708 effort=1 velocity=1 -> lower=-1.5708 upper=1.5708 effort=5.0 velocity=4.0
- joint joint_1B: limit lower=-1.719 upper=3 effort=1 velocity=1 -> lower=-1.719 upper=3 effort=5.0 velocity=4.0
- joint joint_1C: limit lower=-2.4 upper=1.182 effort=1 velocity=1 -> lower=-2.4 upper=1.182 effort=5.0 velocity=4.0
- joint joint_2A: limit lower=-1.5708 upper=1.5708 effort=1 velocity=1 -> lower=-1.5708 upper=1.5708 effort=5.0 velocity=4.0
- joint joint_2B: limit lower=-1.719 upper=3 effort=1 velocity=1 -> lower=-1.719 upper=3 effort=5.0 velocity=4.0
- joint joint_2C: limit lower=-2.4 upper=1.182 effort=1 velocity=1 -> lower=-2.4 upper=1.182 effort=5.0 velocity=4.0
- joint joint_3A: limit lower=-1.5708 upper=1.5708 effort=1 velocity=1 -> lower=-1.5708 upper=1.5708 effort=5.0 velocity=4.0
- joint joint_3B: limit lower=-1.719 upper=3 effort=1 velocity=1 -> lower=-1.719 upper=3 effort=5.0 velocity=4.0
- joint joint_3C: limit lower=-2.4 upper=1.182 effort=1 velocity=1 -> lower=-2.4 upper=1.182 effort=5.0 velocity=4.0
- joint joint_4A: limit lower=-1.5708 upper=1.5708 effort=1 velocity=1 -> lower=-1.5708 upper=1.5708 effort=5.0 velocity=4.0
- joint joint_4B: limit lower=-1.719 upper=3 effort=1 velocity=1 -> lower=-1.719 upper=3 effort=5.0 velocity=4.0
- joint joint_4C: limit lower=-2.4 upper=1.182 effort=1 velocity=1 -> lower=-2.4 upper=1.182 effort=5.0 velocity=4.0
- joint joint_5A: limit lower=-1.5708 upper=1.5708 effort=1 velocity=1 -> lower=-1.5708 upper=1.5708 effort=5.0 velocity=4.0
- joint joint_5B: limit lower=-1.719 upper=3 effort=1 velocity=1 -> lower=-1.719 upper=3 effort=5.0 velocity=4.0
- joint joint_5C: limit lower=-2.4 upper=1.182 effort=1 velocity=1 -> lower=-2.4 upper=1.182 effort=5.0 velocity=4.0
- joint joint_6A: limit lower=-1.5708 upper=1.5708 effort=1 velocity=1 -> lower=-1.5708 upper=1.5708 effort=5.0 velocity=4.0
- joint joint_6B: limit lower=-1.719 upper=3 effort=1 velocity=1 -> lower=-1.719 upper=3 effort=5.0 velocity=4.0
- joint joint_6C: limit lower=-2.4 upper=1.182 effort=1 velocity=1 -> lower=-2.4 upper=1.182 effort=5.0 velocity=4.0

Commit message: Igualar robot a webots: modificacion urdf origin de los joints rpy=000 para que se vea estirado

File: src/dynamixel_hexapod_description/urdf/dynamixel_hexapod.urdf (robot description, URDF)
Before this commit: robot dynamixel_hexapod, 19 links, 18 joints
Joints:
- joint joint_1B: origin xyz=0.07825 0 0 rpy=0.0054103 -0.81909 0.033352 -> xyz=0.07825 0 0 rpy=0 0 0
- joint joint_1C: origin xyz=0.172821824222266 -0.00859357288230811 0 rpy=-3.13913475006377 1.07013691482246 -3.13476958627829 -> xyz=0.172821824222266 -0.00859357288230811 0 rpy=0 0 0
- joint joint_2B: origin xyz=0.0782500731858153 0 0 rpy=0.00541027891423811 -0.819093279009694 0.0333518742125984 -> xyz=0.0782500731858153 0 0 rpy=0 0 0
- joint joint_2C: origin xyz=0.172821824222266 -0.00859357288230778 0 rpy=-3.13913475006377 1.07013691482246 -3.13476958627829 -> xyz=0.172821824222266 -0.00859357288230778 0 rpy=0 0 0
- joint joint_3B: origin xyz=0.0782500731858156 0 0 rpy=0.00541027891423802 -0.819093279009695 0.0333518742125869 -> xyz=0.0782500731858156 0 0 rpy=0 0 0
- joint joint_3C: origin xyz=0.172821824222266 -0.00859357288230712 0 rpy=-3.13913475006378 1.07013691482246 -3.1347695862783 -> xyz=0.172821824222266 -0.00859357288230712 0 rpy=0 0 0
- joint joint_4B: origin xyz=0.0782500731858154 0 0 rpy=0.00541027891423858 -0.819093279009697 0.033351874212595 -> xyz=0.0782500731858154 0 0 rpy=0 0 0
- joint joint_4C: origin xyz=0.172821824222266 -0.00859357288230733 0 rpy=-3.13913475006377 1.07013691482246 -3.13476958627829 -> xyz=0.172821824222266 -0.00859357288230733 0 rpy=0 0 0
- joint joint_5B: origin xyz=0.0782500731858156 0 0 rpy=0.0054102789142378 -0.819093279009694 0.033351874212598 -> xyz=0.0782500731858156 0 0 rpy=0 0 0
- joint joint_5C: origin xyz=0.172821824222266 -0.00859357288230722 0 rpy=-3.13913475006377 1.07013691482246 -3.1347695862783 -> xyz=0.172821824222266 -0.00859357288230722 0 rpy=0 0 0
- joint joint_6B: origin xyz=0.0782500731858157 0 0 rpy=0.00541027891423497 -0.819093279009694 0.0333518742125941 -> xyz=0.0782500731858157 0 0 rpy=0 0 0
- joint joint_6C: origin xyz=0.172821824222266 -0.00859357288230794 0 rpy=-3.13913475006377 1.07013691482246 -3.1347695862783 -> xyz=0.172821824222266 -0.00859357288230794 0 rpy=0 0 0

Commit message: ajuste de limites de los nuevos joints

File: src/dynamixel_hexapod_description/urdf/dynamixel_hexapod.urdf (robot description, URDF)
Before this commit: robot dynamixel_hexapod, 19 links, 18 joints
Joints:
- joint joint_1B: limit lower=-1.719 upper=3 effort=5.0 velocity=4.0 -> lower=-2.5 upper=2.617 effort=5.0 velocity=4.0
- joint joint_1C: limit lower=-2.4 upper=1.182 effort=5.0 velocity=4.0 -> lower=-0.4 upper=3.1 effort=5.0 velocity=4.0
- joint joint_2B: limit lower=-1.719 upper=3 effort=5.0 velocity=4.0 -> lower=-2.5 upper=2.617 effort=5.0 velocity=4.0
- joint joint_2C: limit lower=-2.4 upper=1.182 effort=5.0 velocity=4.0 -> lower=-0.4 upper=3.1 effort=5.0 velocity=4.0
- joint joint_3B: limit lower=-1.719 upper=3 effort=5.0 velocity=4.0 -> lower=-2.5 upper=2.617 effort=5.0 velocity=4.0
- joint joint_3C: limit lower=-2.4 upper=1.182 effort=5.0 velocity=4.0 -> lower=-0.4 upper=3.1 effort=5.0 velocity=4.0
- joint joint_4B: limit lower=-1.719 upper=3 effort=5.0 velocity=4.0 -> lower=-2.5 upper=2.617 effort=5.0 velocity=4.0
- joint joint_4C: limit lower=-2.4 upper=1.182 effort=5.0 velocity=4.0 -> lower=-0.4 upper=3.1 effort=5.0 velocity=4.0
- joint joint_5B: limit lower=-1.719 upper=3 effort=5.0 velocity=4.0 -> lower=-2.5 upper=2.617 effort=5.0 velocity=4.0
- joint joint_5C: limit lower=-2.4 upper=1.182 effort=5.0 velocity=4.0 -> lower=-0.4 upper=3.1 effort=5.0 velocity=4.0
- joint joint_6B: limit lower=-1.719 upper=3 effort=5.0 velocity=4.0 -> lower=-2.5 upper=2.617 effort=5.0 velocity=4.0
- joint joint_6C: limit lower=-2.4 upper=1.182 effort=5.0 velocity=4.0 -> lower=-0.4 upper=3.1 effort=5.0 velocity=4.0
